File: Electronics/multifilament.brd (EAGLE design)
At the start: 68.6 x 53.3 mm, 25 parts, among them IC1 BD6230F, IC2 BD6230F

Commit message: First working version of guillotine software.
Parts:
- C1: device rcl:140CLH-1010 -> rcl:SANYO-OSCON_9F
- moved C1 2.56 mm to (4.76, 25.4)
Routing:
- net +12V: track 48.5 -> 53.2 mm
- net GND: track 90.1 -> 92.5 mm
Changed lines of the file:
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@@
 <element name="R9" library="rcl" package="M0805" value="180R" x="53.34" y="46.6725" rot="R270"/>
 <element name="R10" library="rcl" package="M0805" value="180R" x="55.88" y="46.6725" rot="R270"/>
-<element name="C1" library="rcl" package="140CLH-1010" value="100u" x="6.985" y="26.67" rot="R90"/>
 <element name="I2C" library="pinhead" package="1X04" value="" x="20.0025" y="46.0375"/>
 <element name="//-LEL" library="pinhead" package="1X04" value="" x="64.77" y="11.43" rot="R90"/>
 <element name="C3" library="rcl" package="C0805" value="0.1uF" x="46.6725" y="7.62" rot="R180"/>
 <element name="C5" library="rcl" package="C0805" value="0.1uF" x="15.24" y="41.5925" rot="R90"/>
+<element name="C1" library="rcl" package="SANYO-OSCON_9F" value="100u" x="4.7625" y="25.4" rot="R90"/>
 </elements>
 <signals>
@@
 <contactref element="DRIVE" pad="8"/>
 <contactref element="U$1" pad="GND"/>
-<contactref element="C1" pad="-"/>
 <contactref element="C7" pad="2"/>
 <contactref element="IC2" pad="8"/>
@@
 <contactref element="U$1" pad="GND1"/>
 <contactref element="U$1" pad="GND2"/>
-<wire x1="6.985" y1="22.52" x2="11.4075" y2="22.52" width="0.254" layer="1"/>
 <wire x1="11.4075" y1="22.52" x2="11.43" y2="22.5425" width="0.254" layer="1"/>
 <via x="11.43" y="22.5425" extent="1-16" drill="0.6" diameter="2.54"/>
@@
 <wire x1="58.7375" y1="22.86" x2="59.3725" y2="22.225" width="0.254" layer="1"/>
 <wire x1="59.3725" y1="22.225" x2="59.3725" y2="20.0025" width="0.254" layer="1"/>
+<contactref element="C1" pad="-"/>
+<wire x1="4.7625" y1="22.9" x2="11.0725" y2="22.9" width="0.3048" layer="1"/>
+<wire x1="11.0725" y1="22.9" x2="11.43" y2="22.5425" width="0.3048" layer="1"/>
+<wire x1="16.1925" y1="46.0375" x2="26.416" y2="50.8" width="0" layer="19" extent="1-1"/>
+<wire x1="15.24" y1="42.5425" x2="16.1925" y2="46.0375" width="0" layer="19" extent="1-1"/>
+<wire x1="6.985" y1="39.0525" x2="15.24" y2="42.5425" width="0" layer="19" extent="1-1"/>
+<wire x1="4.7625" y1="22.9" x2="6.985" y2="39.0525" width="0" layer="19" extent="1-1"/>
+<wire x1="38.4175" y1="30.165" x2="34.925" y2="30.165" width="0" layer="19" extent="1-1"/>
+<wire x1="40.8975" y1="29.5275" x2="38.4175" y2="30.165" width="0" layer="19" extent="1-1"/>
+<wire x1="45.7225" y1="7.62" x2="35.8775" y2="14.9225" width="0" layer="19" extent="1-1"/>
+<wire x1="43.18" y1="2.54" x2="45.7225" y2="7.62" width="0" layer="19" extent="1-1"/>
+<wire x1="40.64" y1="2.54" x2="43.18" y2="2.54" width="0" layer="19" extent="1-1"/>
+<wire x1="58.7375" y1="25.0825" x2="40.8975" y2="29.5275" width="0" layer="19" extent="1-16"/>
 </signal>
 <signal name="VIN">
@@
 <contactref element="IC1" pad="6"/>
 <contactref element="C7" pad="1"/>
-<contactref element="C1" pad="+"/>
 <contactref element="IC2" pad="6"/>
 <contactref element="C6" pad="1"/>
@@
 <wire x1="38.4175" y1="32.065" x2="40.895" y2="32.065" width="0.6096" layer="1"/>
 <wire x1="40.895" y1="32.065" x2="40.8975" y2="32.0675" width="0.6096" layer="1"/>
-<wire x1="6.985" y1="36.5125" x2="6.985" y2="30.82" width="1.27" layer="1"/>
-<wire x1="6.985" y1="30.82" x2="10.1825" y2="30.82" width="1.27" layer="1"/>
-<wire x1="10.1825" y1="30.82" x2="11.43" y2="32.0675" width="1.27" layer="1"/>
 <via x="11.43" y="32.0675" extent="1-16" drill="0.6" diameter="2.54"/>
 <wire x1="11.43" y1="32.0675" x2="23.8125" y2="32.0675" width="1.27" layer="16"/>
@@
 <wire x1="23.8125" y1="32.0675" x2="24.4475" y2="32.0675" width="1.27" layer="1"/>
 <wire x1="24.4475" y1="32.0675" x2="26.61" y2="32.0675" width="0.6096" layer="1"/>
+<contactref element="C1" pad="+"/>
+<wire x1="11.43" y1="32.0675" x2="6.985" y2="27.6225" width="1.27" layer="1"/>
+<wire x1="6.985" y1="27.6225" x2="5.04" y2="27.6225" width="1.27" layer="1"/>
+<wire x1="5.04" y1="27.6225" x2="4.7625" y2="27.9" width="1.27" layer="1"/>
+<wire x1="6.985" y1="36.5125" x2="11.43" y2="32.0675" width="1.27" layer="1"/>
+<wire x1="11.7475" y1="31.75" x2="11.43" y2="32.0675" width="1.27" layer="1"/>
 </signal>
 <signal name="+5V">
