File: Electronics/multifilament.sch (EAGLE design)
At the start: 25 parts, among them IC1 BD6230F, IC2 BD6230F

Commit message: First working version of guillotine software.
Parts:
- C1: device rcl:CPOL-EU140CLH-1010 -> rcl:CPOL-EUSANYO_9F
Other:
- note added: "TODO: Make I2C jumper selectable 3V3/5V"
Changed lines of the file:
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@@
 <part name="R10" library="rcl" deviceset="R-EU_" device="M0805" value="180R"/>
 <part name="GND8" library="supply1" deviceset="GND" device=""/>
-<part name="C1" library="rcl" deviceset="CPOL-EU" device="140CLH-1010" value="100u"/>
 <part name="GND9" library="supply1" deviceset="GND" device=""/>
 <part name="I2C" library="pinhead" deviceset="PINHD-1X4" device=""/>
@@
 <part name="GND1" library="supply1" deviceset="GND" device=""/>
 <part name="GND11" library="supply1" deviceset="GND" device=""/>
+<part name="C1" library="rcl" deviceset="CPOL-EU" device="SANYO_9F" value="100u"/>
 </parts>
 <sheets>
@@
 <text x="44.958" y="117.348" size="1.27" layer="95">N.B. Busy is not part of I2C
 But it's useful to the host</text>
+<text x="-33.02" y="127" size="1.778" layer="95">TODO: Make I2C jumper selectable 3V3/5V</text>
 </plain>
 <instances>
@@
 <instance part="R10" gate="G$1" x="101.6" y="15.24"/>
 <instance part="GND8" gate="1" x="15.24" y="10.16"/>
-<instance part="C1" gate="G$1" x="33.02" y="111.76"/>
 <instance part="GND9" gate="1" x="111.76" y="48.26" rot="MR0"/>
 <instance part="I2C" gate="A" x="58.42" y="109.22" rot="R180"/>
@@
 <instance part="GND1" gate="1" x="-5.08" y="45.72"/>
 <instance part="GND11" gate="1" x="17.78" y="48.26"/>
+<instance part="C1" gate="G$1" x="33.02" y="111.76"/>
 </instances>
 <busses>
@@
 <pinref part="GND3" gate="1" pin="GND"/>
 <wire x1="27.94" y1="109.22" x2="27.94" y2="106.68" width="0.1524" layer="91"/>
-<pinref part="C1" gate="G$1" pin="-"/>
 <wire x1="33.02" y1="106.68" x2="27.94" y2="106.68" width="0.1524" layer="91"/>
 <junction x="27.94" y="106.68"/>
+<pinref part="C1" gate="G$1" pin="-"/>
 </segment>
 <segment>
@@
 <wire x1="20.32" y1="111.76" x2="27.94" y2="111.76" width="0.1524" layer="91"/>
 <pinref part="P+1" gate="1" pin="+12V"/>
-<pinref part="C1" gate="G$1" pin="+"/>
 <wire x1="33.02" y1="114.3" x2="27.94" y2="114.3" width="0.1524" layer="91"/>
 <wire x1="27.94" y1="114.3" x2="27.94" y2="111.76" width="0.1524" layer="91"/>
 <junction x="27.94" y="114.3"/>
+<pinref part="C1" gate="G$1" pin="+"/>
 </segment>
 <segment>
